Commit message: Rotate tool0 link to zero

File: kuka_kr6_support/urdf/kr6r900sixx_painter_macro.xacro (robot description, xacro)
@@ -156,5 +156,5 @@
       <parent link="${prefix}link_6"/>
       <child link="${prefix}tool0"/>
-      <origin xyz="0 0 0" rpy="0 ${DEG2RAD * 90} 0"/>
+      <origin xyz="0 0 0" rpy="0 0 0"/>
     </joint>
     <!-- ROS base_link to KUKA $ROBROOT coordinate system transform -->
